Commit message: Gay lord

File: src/joint_description/urdf/joint_model.urdf (robot description, URDF)
Before this commit: robot myfirst, 1 links, 0 joints
Links:
- added link angle_link; visual box size=0.025 0.002 0.002
- added link rotor_link; visual cylinder length=0.010 radius=0.025
- added link stator_link; visual box size=0.102 0.102 0.102
- added link world
- link base_link: geometry 
Joints:
- added joint angle: type revolute, parent stator_link, child rotor_link, origin xyz=0 0 0.056 rpy=0 0 0, axis 0 0 1, limit lower=-3.14159 upper=3.14159 effort=1.0 velocity=3.0
- added joint base_joint: type fixed, parent world, child base_link, origin xyz=0 0 0 rpy=0 0 0
- added joint indicator: type fixed, parent rotor_link, child angle_link, origin xyz=0.0125 0 0.006 rpy=0 0 0
- added joint stator_joint: type fixed, parent base_link, child stator_link, origin xyz=0 0 0.051 rpy=0 0 0

Commit message: funny

File: src/joint_description/urdf/joint_model.urdf (robot description, URDF)
Before this commit: robot joint_model, 5 links, 4 joints
Links:
- link angle_link: mass None -> 0.1; geometry collision box size=${angle_length} ${angle_width} ${angle_height}; visual box size=${angle_length} ${angle_width} ${angle_height}
- link base_link: mass None -> 0.1
- link rotor_link: mass None -> 0.5; geometry collision cylinder length=${rotor_height} radius=${rotor_radius}; visual cylinder length=${rotor_height} radius=${rotor_radius}
- link stator_link: mass None -> 1.0; geometry collision box size=${stator_size} ${stator_size} ${stator_size}; visual box size=${stator_size} ${stator_size} ${stator_size}
Joints:
- joint angle: origin xyz=0 0 0.056 rpy=0 0 0 -> xyz=0 0 ${stator_half + rotor_half} rpy=0 0 0
- joint indicator: origin xyz=0.0125 0 0.006 rpy=0 0 0 -> xyz=${rotor_radius/2} 0 ${rotor_half + 1*mm} rpy=0 0 0
- joint stator_joint: origin xyz=0 0 0.051 rpy=0 0 0 -> xyz=0 0 ${stator_half} rpy=0 0 0

Commit message: Stor KUK

File: src/joint_description/urdf/joint_model.urdf (robot description, URDF)
Before this commit: robot joint_model, 5 links, 4 joints
Links:
- removed link angle_link
- removed link base_link
- removed link rotor_link
- removed link stator_link
- link world: mass None -> 1.0
Joints:
- removed joint angle
- removed joint indicator
- removed joint stator_joint
- joint base_joint: child base_link -> ur1_base_link
